File: Platine/Gemeine Platine/AbuDhabi_ElectronBeam.kicad_sch (KiCad schematic)
At the start: 22 parts, among them J1 Comms, J12 Sensor, J13 Bomba, J16 Power, J18 Buttons, J2 Opt. ext. Ausgangsspannung, J3 Opt. Ard. Ausgangspannung, U1 74LS01, U6 74LS20

Commit message: Small change in schematic
Parts:
- U1: value 74LS01 -> MM74H0M
Changed lines of the file:
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@@
       (effects (font (size 1.27 1.27)))
     )
-    (property "Value" "74LS01" (at 155.5115 102.87 0)
+    (property "Value" "MM74H0M" (at 155.5115 102.87 0)
       (effects (font (size 1.27 1.27)))
     )
