File: Platine/Neue_Pumpe/Final_PCB/Signal_cond.kicad_sch (KiCad schematic)
At the start: 78 parts

Commit message: final PCB finished
Parts:
- removed C19: 100n, Capacitor_SMD:C_0603_1608Metric_Pad1.08x0.95mm_HandSolder, symbol Device:C
Changed lines of the file:
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@@
 	)
 	(junction
-		(at 218.44 39.37)
-		(diameter 0)
-		(color 0 0 0 0)
-	)
-	(junction
 		(at 177.8 96.52)
 		(diameter 0)
@@
 	(wire
 		(pts
-			(xy 231.14 39.37) (xy 218.44 39.37)
+			(xy 231.14 39.37) (xy 220.98 39.37)
 		)
 		(stroke
@@
 	(wire
 		(pts
-			(xy 218.44 39.37) (xy 218.44 38.1)
+			(xy 220.98 39.37) (xy 220.98 38.1)
 		)
 		(stroke
@@
 	(wire
 		(pts
-			(xy 218.44 49.53) (xy 218.44 50.8)
-		)
-		(stroke
-			(width 0)
-			(type default)
-		)
-	)
-	(wire
-		(pts
 			(xy 26.67 135.89) (xy 26.67 137.16)
 		)
@@
 	(wire
 		(pts
-			(xy 218.44 39.37) (xy 218.44 41.91)
-		)
-		(stroke
-			(width 0)
-			(type default)
-		)
-	)
-	(wire
-		(pts
 			(xy 265.43 39.37) (xy 275.59 39.37)
 		)
@@
 	(symbol
 		(lib_id "power:GNDD")
-		(at 218.44 50.8 0)
-		(unit 1)
-		(exclude_from_sim no)
-		(in_bom yes)
-		(on_board yes)
-		(dnp no)
-		(fields_autoplaced yes)
-		(property "Reference" "#PWR038"
-			(at 218.44 57.15 0)
-			(effects
-				(font
-					(size 1.27 1.27)
-				)
-				(hide yes)
-			)
-		)
-		(property "Value" "GNDD"
-			(at 218.44 54.61 0)
-			(effects
-				(font
-					(size 1.27 1.27)
-				)
-			)
-		)
-		(property "Footprint" ""
-			(at 218.44 50.8 0)
-			(effects
-				(font
-					(size 1.27 1.27)
-				)
-				(hide yes)
-			)
-		)
-		(property "Datasheet" ""
-			(at 218.44 50.8 0)
-			(effects
-				(font
-					(size 1.27 1.27)
-				)
-				(hide yes)
-			)
-		)
-		(property "Description" "Power symbol creates a global label with name \"GNDD\" , digital ground"
-			(at 218.44 50.8 0)
-			(effects
-				(font
-					(size 1.27 1.27)
-				)
-				(hide yes)
-			)
-		)
-		(pin "1"
-		)
-		(instances
-			(project "Final_PCB"
-				(path "/160fd78b-052f-42a7-9b7c-961e371280e5/1bce4860-ff53-4a06-a9be-ec3e27221410"
-					(reference "#PWR038")
-					(unit 1)
-				)
-			)
-		)
-	)
-	(symbol
-		(lib_id "power:GNDD")
 		(at 41.91 106.68 0)
 		(unit 1)
@@
 	(symbol
 		(lib_id "Device:C")
-		(at 218.44 45.72 0)
-		(mirror x)
-		(unit 1)
-		(exclude_from_sim no)
-		(in_bom yes)
-		(on_board yes)
-		(dnp no)
-		(property "Reference" "C19"
-			(at 214.63 44.4499 0)
-			(effects
-				(font
-					(size 1.27 1.27)
-				)
-				(justify right)
-			)
-		)
-		(property "Value" "100n"
-			(at 214.63 46.9899 0)
-			(effects
-				(font
-					(size 1.27 1.27)
-				)
-				(justify right)
-			)
-		)
-		(property "Footprint" "Capacitor_SMD:C_0603_1608Metric_Pad1.08x0.95mm_HandSolder"
-			(at 219.4052 41.91 0)
-			(effects
-				(font
-					(size 1.27 1.27)
-				)
-				(hide yes)
-			)
-		)
-		(property "Datasheet" "~"
-			(at 218.44 45.72 0)
-			(effects
-				(font
-					(size 1.27 1.27)
-				)
-				(hide yes)
-			)
-		)
-		(property "Description" "Unpolarized capacitor"
-			(at 218.44 45.72 0)
-			(effects
-				(font
-					(size 1.27 1.27)
-				)
-				(hide yes)
-			)
-		)
-		(pin "2"
-		)
-		(pin "1"
-		)
-		(instances
-			(project "Final_PCB"
-				(path "/160fd78b-052f-42a7-9b7c-961e371280e5/1bce4860-ff53-4a06-a9be-ec3e27221410"
-					(reference "C19")
-					(unit 1)
-				)
-			)
-		)
-	)
-	(symbol
-		(lib_id "Device:C")
 		(at 219.71 92.71 0)
 		(mirror x)
@@
 		(lib_name "+3.3V_1")
 		(lib_id "power:+3.3V")
-		(at 218.44 38.1 0)
+		(at 220.98 38.1 0)
 		(unit 1)
 		(exclude_from_sim no)
@@
 		(dnp no)
 		(property "Reference" "#PWR037"
-			(at 218.44 41.91 0)
+			(at 220.98 41.91 0)
 			(effects
 				(font
@@
 		)
 		(property "Value" "+3.3VD"
-			(at 216.154 34.544 0)
+			(at 218.694 34.544 0)
 			(effects
 				(font
@@
 		)
 		(property "Footprint" ""
-			(at 218.44 38.1 0)
+			(at 220.98 38.1 0)
 			(effects
 				(font
@@
 		)
 		(property "Datasheet" ""
-			(at 218.44 38.1 0)
+			(at 220.98 38.1 0)
 			(effects
 				(font
@@
 		)
 		(property "Description" "Power symbol creates a global label with name \"+3.3V\""
-			(at 218.44 38.1 0)
+			(at 220.98 38.1 0)
 			(effects
 				(font
