File: Platine/Neue_Pumpe/Final_PCB/sensors.kicad_sch (KiCad schematic)
At the start: 27 parts

Commit message: a lot of advance in final PCB
Connections:
- net analog_inp_7: no longer U12.2 (AIP), U13.2 (AIP)
- new net analog_inp_8: U12.2 (AIP)
- new net analog_inp_9: U13.2 (AIP)
Changed lines of the file:
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@@
 		)
 	)
-	(label "analog_inp_8"
+	(label "analog_inp_7"
 		(at 214.63 45.72 0)
 		(fields_autoplaced yes)
@@
 		)
 	)
-	(label "analog_inp_10"
+	(label "analog_inp_9"
 		(at 214.63 53.34 0)
 		(fields_autoplaced yes)
@@
 		)
 	)
-	(label "analog_inp_9"
+	(label "analog_inp_8"
 		(at 214.63 49.53 0)
 		(fields_autoplaced yes)

Commit message: final PCB finished
Parts:
- removed C26, C33: 0.1uF, Capacitor_SMD:C_0603_1608Metric_Pad1.08x0.95mm_HandSolder, symbol Device:C
Other:
- moved on the sheet: C28, C30, C31, C32, C34, C35
